Commit message: style

File: tests/output.urdf (robot description, URDF)
Before this commit: robot vgc10_extender_stick, 6 links, 5 joints
Links:
- link CONNECTED:OUTPUT-vgc10_extender_stick: mass 0 -> None
- link CONNECTED:OUTPUT-vgc10_extender_stick(1): mass 0 -> None
- link OUTPUT-vgc10_extender_stick: mass 0 -> None
